File: hardware/cdp-mobo/cdp-oscillator.kicad_sch (KiCad schematic)
At the start: 8 parts, among them U9 74HC00, Y1 2MHz

Commit message: Minor changes in component values, and added a the IO module.
Parts:
- Y1: value 2MHz -> 2.4576MHz
Other:
- moved on the sheet: U9D
Changed lines of the file:
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@@
   (junction (at 156.21 105.41) (diameter 0) (color 0 0 0 0)
   )
-  (junction (at 189.865 97.155) (diameter 0) (color 0 0 0 0)
+  (junction (at 189.865 97.79) (diameter 0) (color 0 0 0 0)
   )
   (junction (at 144.78 82.55) (diameter 0) (color 0 0 0 0)
@@
     (stroke (width 0) (type default))
   )
-  (wire (pts (xy 189.865 97.155) (xy 191.135 97.155))
+  (wire (pts (xy 189.865 97.79) (xy 191.135 97.79))
     (stroke (width 0) (type default))
   )
@@
     (stroke (width 0) (type default))
   )
-  (wire (pts (xy 189.865 92.075) (xy 191.135 92.075))
-    (stroke (width 0) (type default))
-  )
-  (wire (pts (xy 189.865 92.075) (xy 189.865 97.155))
+  (wire (pts (xy 189.865 92.71) (xy 191.135 92.71))
+    (stroke (width 0) (type default))
+  )
+  (wire (pts (xy 189.865 92.71) (xy 189.865 97.79))
     (stroke (width 0) (type default))
   )
@@
     (stroke (width 0) (type default))
   )
-  (wire (pts (xy 189.865 97.155) (xy 189.865 100.33))
+  (wire (pts (xy 189.865 97.79) (xy 189.865 100.965))
     (stroke (width 0) (type default))
   )
@@
     )
   )
-  (symbol (lib_id "power:GND") (at 189.865 100.33 0) (unit 1)
-    (in_bom yes) (on_board yes) (dnp no) (fields_autoplaced)
-    (property "Reference" "#PWR034" (at 189.865 106.68 0)
-      (effects (font (size 1.27 1.27)) hide)
-    )
-    (property "Value" "GND" (at 189.865 105.41 0)
-      (effects (font (size 1.27 1.27)))
-    )
-    (property "Footprint" "" (at 189.865 100.33 0)
-      (effects (font (size 1.27 1.27)) hide)
-    )
-    (property "Datasheet" "" (at 189.865 100.33 0)
+  (symbol (lib_id "power:GND") (at 189.865 100.965 0) (unit 1)
+    (in_bom yes) (on_board yes) (dnp no) (fields_autoplaced)
+    (property "Reference" "#PWR034" (at 189.865 107.315 0)
+      (effects (font (size 1.27 1.27)) hide)
+    )
+    (property "Value" "GND" (at 189.865 106.045 0)
+      (effects (font (size 1.27 1.27)))
+    )
+    (property "Footprint" "" (at 189.865 100.965 0)
+      (effects (font (size 1.27 1.27)) hide)
+    )
+    (property "Datasheet" "" (at 189.865 100.965 0)
       (effects (font (size 1.27 1.27)) hide)
     )
@@
       (effects (font (size 1.27 1.27)))
     )
-    (property "Value" "2MHz" (at 156.21 88.9 0)
+    (property "Value" "2.4576MHz" (at 156.21 88.9 0)
       (effects (font (size 1.27 1.27)))
     )
@@
     )
   )
-  (symbol (lib_id "74xx:74LS00") (at 198.755 94.615 0) (unit 4)
-    (in_bom yes) (on_board yes) (dnp no) (fields_autoplaced)
-    (property "Reference" "U9" (at 198.7467 86.995 0)
-      (effects (font (size 1.27 1.27)))
-    )
-    (property "Value" "74HC00" (at 198.7467 89.535 0)
-      (effects (font (size 1.27 1.27)))
-    )
-    (property "Footprint" "Package_DIP:DIP-14_W7.62mm_Socket" (at 198.755 94.615 0)
-      (effects (font (size 1.27 1.27)) hide)
-    )
-    (property "Datasheet" "http://www.ti.com/lit/gpn/sn74ls00" (at 198.755 94.615 0)
-      (effects (font (size 1.27 1.27)) hide)
-    )
+  (symbol (lib_id "74xx:74LS00") (at 198.755 95.25 0) (unit 4)
+    (in_bom yes) (on_board yes) (dnp no) (fields_autoplaced)
+    (property "Reference" "U9" (at 198.7467 87.63 0)
+      (effects (font (size 1.27 1.27)))
+    )
+    (property "Value" "74HC00" (at 198.7467 90.17 0)
+      (effects (font (size 1.27 1.27)))
+    )
+    (property "Footprint" "Package_DIP:DIP-14_W7.62mm_Socket" (at 198.755 95.25 0)
+      (effects (font (size 1.27 1.27)) hide)
+    )
+    (property "Datasheet" "http://www.ti.com/lit/gpn/sn74ls00" (at 198.755 95.25 0)
+      (effects (font (size 1.27 1.27)) hide)
+    )
