File: hardware/cdp-io/cdp-io.kicad_sch (KiCad schematic)
At the start: 0 parts

Commit message: Added the controller page, and two decoders are placed in it. Moved some files, and added the gitignore file.
Other:
- added sheet Controller (cdp-controller.kicad_sch)
Changed lines of the file:
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@@
+    )
+  )
+  (sheet (at 200.66 33.02) (size 40.005 21.59) (fields_autoplaced)
+    (stroke (width 0.1524) (type solid))
+    (fill (color 0 0 0 0.0000))
+    (property "Sheetname" "Controller" (at 200.66 32.3084 0)
+      (effects (font (size 1.27 1.27)) (justify left bottom))
+    )
+    (property "Sheetfile" "cdp-controller.kicad_sch" (at 200.66 55.1946 0)
+      (effects (font (size 1.27 1.27)) (justify left top))
+    )
+    (instances
+      (project "cdp-io"
+        (path "/479e9a3e-8705-41df-8009-7e8503809f49" (page "6"))
+      )
     )
   )

Commit message: The final version of the IO board. Gerber files added.
Other:
- company: (none) -> ZLED
- title: (none) -> Root
Changed lines of the file:
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@@
 (kicad_sch (version 20230121) (generator eeschema)
   (paper "A4")
+  (title_block
+    (title "Root")
+    (date "2023-07-06")
+    (rev "1")
+    (company "ZLED")
+  )
   (sheet (at 115.57 33.02) (size 40.005 21.59) (fields_autoplaced)
     (stroke (width 0.1524) (type solid))
