File: hardware/cdp-io/cdp-controller.kicad_sch (KiCad schematic)
At the start: 6 parts, among them U7 74LS00, U8 74LS138, U9 74LS138

Commit message: The controller is finished. U7 is changed to a hex inverter.
Parts:
- removed U7: 74LS00, symbol 74xx:74LS00
- added C1: 100n, Capacitor_THT:C_Disc_D3.0mm_W1.6mm_P2.50mm, symbol Device:C_Small
- added U10: 74LS175, symbol 74xx:74LS175
- added U7: 74LS14, symbol 74xx:74LS14
Connections:
- net GND: now also C1.2, U10.8 (GND), U7.7 (GND)
- net TPB: now also U7.9
- net VCC: now also C1.1, U10.16 (VCC), U7.14 (VCC)
- net at U8.4 (E1), U9.4 (E1): now also U7.8
- net ~{PORTC WRITE}: now reaches U8.11 (O4)
- net ~{PORTB WRITE}: now reaches U8.12 (O3)
- net ~{PORTA WRITE}: now reaches U8.13 (O2)
- net ~{CTRL WRITE}: now reaches U8.14 (O1)
- net ~{CTRL WRITE}: now also U7.11
- net ~{PORTC READ}: now reaches U9.11 (O4)
- net ~{PORTB READ}: now reaches U9.12 (O3)
- net ~{PORTA READ}: now reaches U9.13 (O2)
- new net: U10.9 (Cp), U7.10
- new net D0: U10.4 (D0)
- new net D1: U10.5 (D1)
- new net D2: U10.12 (D2)
- new net D3: U10.13 (D3)
- new net ~{PORTA OUTPUT}: U10.3 (~{Q0})
- new net ~{PORTB OUTPUT}: U10.6 (~{Q1})
- new net ~{PORTC OUTPUT}: U10.11 (~{Q2})
- new net ~{RESET}: U10.1 (~{Mr})

Commit message: Changed the layout a bit, started to work on the PCB.
Parts:
- U10, U8, U9: footprint (none) -> Package_DIP:DIP-16_W7.62mm_Socket
- U7: footprint (none) -> Package_DIP:DIP-14_W7.62mm_Socket
Other:
- moved on the sheet: C1

Commit message: Changed the schematic a bit.
Parts:
- removed unit 4 of U7
- removed unit 6 of U7
- removed unit 5 of U7
- added unit 1 of U7
- added unit 2 of U7
- added unit 3 of U7
Connections:
- net D1: now also U10.12 (D2); no longer U10.5 (D1)
- net D2: now also U10.13 (D3); no longer U10.12 (D2)
- net D3: now also U10.5 (D1); no longer U10.13 (D3)
- net TPB: now also U7.5
- net ~{CTRL WRITE}: now also U7.3
- net ~{PORTB OUTPUT}: now also U10.11 (~{Q2}); no longer U10.6 (~{Q1})
- net ~{PORTC OUTPUT}: now also U10.14 (~{Q3}); no longer U10.11 (~{Q2})
- net at U8.4 (E1), U9.4 (E1): now also U7.6
- net at U10.9 (Cp): now also U7.4

Commit message: A really small progress.
Connections:
- net D0: now also U10.13 (D3); no longer U10.4 (D0)
- net D2: now also U10.5 (D1); no longer U10.13 (D3)
- net D3: now also U10.4 (D0); no longer U10.5 (D1)
- net ~{CTRL WRITE}: now also U7.1; no longer U7.3
- net ~{PORTA OUTPUT}: now also U10.14 (~{Q3}); no longer U10.3 (~{Q0})
- net ~{PORTC OUTPUT}: now also U10.6 (~{Q1}); no longer U10.14 (~{Q3})
- net at U7.2: now also U10.9 (Cp)
- net at U7.4: no longer U10.9 (Cp)
- net ~{MRW} renamed ~{MWR}
Other:
- moved on the sheet: U7A, U7B

Commit message: Renamed a few net, and changed the schematic a bit. The PCB is ready!
Parts:
- added R1, R2: 47k, Resistor_THT:R_Axial_DIN0207_L6.3mm_D2.5mm_P10.16mm_Horizontal, symbol Device:R_Small
Connections:
- net GND: now also R1.2, R2.2
- net TPB: now also R1.1
- net ~{RESET} renamed ~{CLEAR}
- net ~{CLEAR}: now also R2.1
Changed lines of the file:
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@@
   (junction (at 113.03 47.625) (diameter 0) (color 0 0 0 0)
   )
+  (junction (at 95.25 105.41) (diameter 0) (color 0 0 0 0)
+  )
+  (junction (at 95.25 171.45) (diameter 0) (color 0 0 0 0)
+  )
   (junction (at 116.205 105.41) (diameter 0) (color 0 0 0 0)
   )
@@
     (stroke (width 0) (type default))
   )
-  (wire (pts (xy 90.805 105.41) (xy 97.155 105.41))
+  (wire (pts (xy 85.725 105.41) (xy 95.25 105.41))
     (stroke (width 0) (type default))
   )
@@
     (stroke (width 0) (type default))
   )
+  (wire (pts (xy 95.25 171.45) (xy 95.25 173.99))
+    (stroke (width 0) (type default))
+  )
   (wire (pts (xy 125.095 92.71) (xy 125.095 40.005))
     (stroke (width 0) (type default))
@@
     (stroke (width 0) (type default))
   )
+  (wire (pts (xy 95.25 113.665) (xy 95.25 115.57))
+    (stroke (width 0) (type default))
+  )
   (wire (pts (xy 116.205 52.705) (xy 116.205 105.41))
     (stroke (width 0) (type default))
@@
     (stroke (width 0) (type default))
   )
+  (wire (pts (xy 95.25 171.45) (xy 123.19 171.45))
+    (stroke (width 0) (type default))
+  )
   (wire (pts (xy 113.665 164.465) (xy 120.65 164.465))
     (stroke (width 0) (type default))
@@
     (stroke (width 0) (type default))
   )
+  (wire (pts (xy 95.25 108.585) (xy 95.25 105.41))
+    (stroke (width 0) (type default))
+  )
   (wire (pts (xy 142.875 22.225) (xy 142.875 26.035))
     (stroke (width 0) (type default))
@@
     (stroke (width 0) (type default))
   )
-  (wire (pts (xy 90.805 171.45) (xy 123.19 171.45))
+  (wire (pts (xy 90.805 171.45) (xy 95.25 171.45))
     (stroke (width 0) (type default))
   )
@@
     (stroke (width 0) (type default))
   )
+  (wire (pts (xy 95.25 181.61) (xy 95.25 179.07))
+    (stroke (width 0) (type default))
+  )
   (wire (pts (xy 90.805 34.925) (xy 127.635 34.925))
     (stroke (width 0) (type default))
@@
     (stroke (width 0) (type default))
   )
+  (wire (pts (xy 95.25 105.41) (xy 97.155 105.41))
+    (stroke (width 0) (type default))
+  )
   (wire (pts (xy 132.715 26.035) (xy 135.89 26.035))
     (stroke (width 0) (type default))
@@
     (stroke (width 0) (type default))
   )
-  (global_label "TPB" (shape input) (at 90.805 105.41 180) (fields_autoplaced)
+  (global_label "TPB" (shape input) (at 85.725 105.41 180) (fields_autoplaced)
     (effects (font (size 1.27 1.27)) (justify right))
-    (property "Intersheetrefs" "${INTERSHEET_REFS}" (at 84.3916 105.41 0)
+    (property "Intersheetrefs" "${INTERSHEET_REFS}" (at 79.3116 105.41 0)
       (effects (font (size 1.27 1.27)) (justify right) hide)
     )
@@
     )
   )
-  (global_label "~{RESET}" (shape input) (at 90.805 171.45 180) (fields_autoplaced)
+  (global_label "~{CLEAR}" (shape input) (at 90.805 171.45 180) (fields_autoplaced)
     (effects (font (size 1.27 1.27)) (justify right))
-    (property "Intersheetrefs" "${INTERSHEET_REFS}" (at 82.1541 171.45 0)
+    (property "Intersheetrefs" "${INTERSHEET_REFS}" (at 82.0935 171.45 0)
       (effects (font (size 1.27 1.27)) (justify right) hide)
     )
@@
     )
   )
+  (symbol (lib_id "Device:R_Small") (at 95.25 176.53 0) (unit 1)
+    (in_bom yes) (on_board yes) (dnp no) (fields_autoplaced)
+    (property "Reference" "R2" (at 97.79 175.895 0)
+      (effects (font (size 1.27 1.27)) (justify left))
+    )
+    (property "Value" "47k" (at 97.79 178.435 0)
+      (effects (font (size 1.27 1.27)) (justify left))
+    )
+    (property "Footprint" "Resistor_THT:R_Axial_DIN0207_L6.3mm_D2.5mm_P10.16mm_Horizontal" (at 95.25 176.53 0)
+      (effects (font (size 1.27 1.27)) hide)
+    )
+    (property "Datasheet" "~" (at 95.25 176.53 0)
+      (effects (font (size 1.27 1.27)) hide)
+    )
+    (pin "1")
+    (pin "2")
+    (instances
+      (project "cdp-io"
+        (path "/479e9a3e-8705-41df-8009-7e8503809f49/fc5dd19a-450f-4ce7-af21-025e7154e993"
+          (reference "R2") (unit 1)
+        )
+      )
+    )
+  )
   (symbol (lib_id "74xx:74LS138") (at 142.875 95.25 0) (unit 1)
     (in_bom yes) (on_board yes) (dnp no) (fields_autoplaced)
@@
     )
   )
+  (symbol (lib_id "Device:R_Small") (at 95.25 111.125 0) (unit 1)
+    (in_bom yes) (on_board yes) (dnp no) (fields_autoplaced)
+    (property "Reference" "R1" (at 97.79 110.49 0)
+      (effects (font (size 1.27 1.27)) (justify left))
+    )
+    (property "Value" "47k" (at 97.79 113.03 0)
+      (effects (font (size 1.27 1.27)) (justify left))
+    )
+    (property "Footprint" "Resistor_THT:R_Axial_DIN0207_L6.3mm_D2.5mm_P10.16mm_Horizontal" (at 95.25 111.125 0)
+      (effects (font (size 1.27 1.27)) hide)
+    )
+    (property "Datasheet" "~" (at 95.25 111.125 0)
+      (effects (font (size 1.27 1.27)) hide)
+    )
+    (pin "1")
+    (pin "2")
+    (instances
+      (project "cdp-io"
+        (path "/479e9a3e-8705-41df-8009-7e8503809f49/fc5dd19a-450f-4ce7-af21-025e7154e993"
+          (reference "R1") (unit 1)
+        )
+      )
+    )
+  )
   (symbol (lib_id "Device:C_Small") (at 138.43 78.74 270) (unit 1)
     (in_bom yes) (on_board yes) (dnp no) (fields_autoplaced)
@@
         (path "/479e9a3e-8705-41df-8009-7e8503809f49/03dab4a8-d44b-4cf8-b119-6efcff8953b4"
           (reference "U7") (unit 3)
+        )
+      )
+    )
+  )
+  (symbol (lib_id "power:GND") (at 95.25 181.61 0) (unit 1)
+    (in_bom yes) (on_board yes) (dnp no) (fields_autoplaced)
+    (property "Reference" "#PWR04" (at 95.25 187.96 0)
+      (effects (font (size 1.27 1.27)) hide)
+    )
+    (property "Value" "GND" (at 95.25 186.055 0)
+      (effects (font (size 1.27 1.27)))
+    )
+    (property "Footprint" "" (at 95.25 181.61 0)
+      (effects (font (size 1.27 1.27)) hide)
+    )
+    (property "Datasheet" "" (at 95.25 181.61 0)
+      (effects (font (size 1.27 1.27)) hide)
+    )
+    (pin "1")
+    (instances
+      (project "cdp-io"
+        (path "/479e9a3e-8705-41df-8009-7e8503809f49"
+          (reference "#PWR04") (unit 1)
+        )
+        (path "/479e9a3e-8705-41df-8009-7e8503809f49/05095c2f-eeee-4b53-a55c-38329025afd6"
+          (reference "#PWR06") (unit 1)
+        )
+        (path "/479e9a3e-8705-41df-8009-7e8503809f49/f2f2e87f-81b0-49e1-b285-4bb1f98f04a0"
+          (reference "#PWR02") (unit 1)
+        )
+        (path "/479e9a3e-8705-41df-8009-7e8503809f49/fc5dd19a-450f-4ce7-af21-025e7154e993"
+          (reference "#PWR042") (unit 1)
         )
       )
@@
         )
       )
+    )
+  )
+  (symbol (lib_id "power:GND") (at 95.25 115.57 0) (unit 1)
+    (in_bom yes) (on_board yes) (dnp no) (fields_autoplaced)
+    (property "Reference" "#PWR04" (at 95.25 121.92 0)
+      (effects (font (size 1.27 1.27)) hide)
+    )
+    (property "Value" "GND" (at 95.25 120.015 0)
+      (effects (font (size 1.27 1.27)))
+    )
+    (property "Footprint" "" (at 95.25 115.57 0)
+      (effects (font (size 1.27 1.27)) hide)
+    )
+    (property "Datasheet" "" (at 95.25 115.57 0)
+      (effects (font (size 1.27 1.27)) hide)
+    )
+    (pin "1")
+    (instances
+      (project "cdp-io"
+        (path "/479e9a3e-8705-41df-8009-7e8503809f49"
+          (reference "#PWR04") (unit 1)
+        )
+        (path "/479e9a3e-8705-41df-8009-7e8503809f49/05095c2f-eeee-4b53-a55c-38329025afd6"
+          (reference "#PWR06") (unit 1)
+        )
+        (path "/479e9a3e-8705-41df-8009-7e8503809f49/f2f2e87f-81b0-49e1-b285-4bb1f98f04a0"
+          (reference "#PWR02") (unit 1)
+        )
+        (path "/479e9a3e-8705-41df-8009-7e8503809f49/fc5dd19a-450f-4ce7-af21-025e7154e993"
+          (reference "#PWR041") (unit 1)
+        )
+      )

Commit message: The final version of the IO board. Gerber files added.
Connections:
- net GND: now also U7.3
Other:
- company: (none) -> ZLED
- title: (none) -> Controller
- moved on the sheet: U7B
Changed lines of the file:
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@@
 (kicad_sch (version 20230121) (generator eeschema)
   (paper "A4")
+  (title_block
+    (title "Controller")
+    (date "2023-07-06")
+    (rev "1")
+    (company "ZLED")
+  )
   (junction (at 127.635 34.925) (diameter 0) (color 0 0 0 0)
   )
@@
     (stroke (width 0) (type default))
   )
+  (wire (pts (xy 36.83 127.635) (xy 36.83 128.905))
+    (stroke (width 0) (type default))
+  )
   (wire (pts (xy 130.175 90.17) (xy 126.365 90.17))
     (stroke (width 0) (type default))
@@
   )
   (wire (pts (xy 90.805 171.45) (xy 95.25 171.45))
+    (stroke (width 0) (type default))
+  )
+  (wire (pts (xy 38.1 127.635) (xy 36.83 127.635))
     (stroke (width 0) (type default))
   )
@@
     )
   )
+  (symbol (lib_id "power:GND") (at 36.83 128.905 0) (unit 1)
+    (in_bom yes) (on_board yes) (dnp no) (fields_autoplaced)
+    (property "Reference" "#PWR04" (at 36.83 135.255 0)
+      (effects (font (size 1.27 1.27)) hide)
+    )
+    (property "Value" "GND" (at 36.83 133.35 0)
+      (effects (font (size 1.27 1.27)))
+    )
+    (property "Footprint" "" (at 36.83 128.905 0)
+      (effects (font (size 1.27 1.27)) hide)
+    )
+    (property "Datasheet" "" (at 36.83 128.905 0)
+      (effects (font (size 1.27 1.27)) hide)
+    )
+    (pin "1")
+    (instances
+      (project "cdp-io"
+        (path "/479e9a3e-8705-41df-8009-7e8503809f49"
+          (reference "#PWR04") (unit 1)
+        )
+        (path "/479e9a3e-8705-41df-8009-7e8503809f49/05095c2f-eeee-4b53-a55c-38329025afd6"
+          (reference "#PWR06") (unit 1)
+        )
+        (path "/479e9a3e-8705-41df-8009-7e8503809f49/f2f2e87f-81b0-49e1-b285-4bb1f98f04a0"
+          (reference "#PWR02") (unit 1)
+        )
+        (path "/479e9a3e-8705-41df-8009-7e8503809f49/fc5dd19a-450f-4ce7-af21-025e7154e993"
+          (reference "#PWR044") (unit 1)
+        )
+      )
+    )
+  )
   (symbol (lib_id "Device:R_Small") (at 95.25 176.53 0) (unit 1)
     (in_bom yes) (on_board yes) (dnp no) (fields_autoplaced)
@@
     )
   )
-  (symbol (lib_id "74xx:74LS14") (at 60.96 133.35 0) (unit 2)
-    (in_bom yes) (on_board yes) (dnp no) (fields_autoplaced)
-    (property "Reference" "U7" (at 60.96 125.095 0)
-      (effects (font (size 1.27 1.27)))
-    )
-    (property "Value" "74LS14" (at 60.96 127.635 0)
-      (effects (font (size 1.27 1.27)))
-    )
-    (property "Footprint" "Package_DIP:DIP-14_W7.62mm_Socket" (at 60.96 133.35 0)
-      (effects (font (size 1.27 1.27)) hide)
-    )
-    (property "Datasheet" "http://www.ti.com/lit/gpn/sn74LS14" (at 60.96 133.35 0)
-      (effects (font (size 1.27 1.27)) hide)
-    )
+  (symbol (lib_id "74xx:74LS14") (at 45.72 127.635 0) (unit 2)
+    (in_bom yes) (on_board yes) (dnp no) (fields_autoplaced)
+    (property "Reference" "U7" (at 45.72 119.38 0)
+      (effects (font (size 1.27 1.27)))
+    )
+    (property "Value" "74LS14" (at 45.72 121.92 0)
+      (effects (font (size 1.27 1.27)))
+    )
+    (property "Footprint" "Package_DIP:DIP-14_W7.62mm_Socket" (at 45.72 127.635 0)
+      (effects (font (size 1.27 1.27)) hide)
+    )
+    (property "Datasheet" "http://www.ti.com/lit/gpn/sn74LS14" (at 45.72 127.635 0)
+      (effects (font (size 1.27 1.27)) hide)
+    )
