File: hardware/cdp-leddriver/cdp-stepper.kicad_sch (KiCad schematic)
At the start: 7 parts, among them U5 74LS74, U6 74LS132, U7 74LS74

Commit message: IC names fixed on the led driver schematic, on the PCB the MA8-MA15 labels were misaligned that is also fixed. Updated the gerber files.
Parts:
- U5, U7: value 74LS74 -> 74HC74
- U6: value 74LS132 -> 74HC132
- U6: value 74LS132 -> 74HC132; footprint (none) -> Package_DIP:DIP-14_W7.62mm_Socket
Changed lines of the file:
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@@
       (effects (font (size 1.27 1.27)) (justify left))
     )
-    (property "Value" "74LS74" (at 194.945 43.18 0)
+    (property "Value" "74HC74" (at 194.945 43.18 0)
       (effects (font (size 1.27 1.27)) (justify left))
     )
@@
       (effects (font (size 1.27 1.27)))
     )
-    (property "Value" "74LS132" (at 128.2617 48.26 0)
+    (property "Value" "74HC132" (at 128.2617 48.26 0)
       (effects (font (size 1.27 1.27)))
     )
@@
       (effects (font (size 1.27 1.27)) (justify left))
     )
-    (property "Value" "74LS132" (at 259.08 43.18 0)
+    (property "Value" "74HC132" (at 259.08 43.18 0)
       (effects (font (size 1.27 1.27)) (justify left))
     )
@@
       (effects (font (size 1.27 1.27)))
     )
-    (property "Value" "74LS132" (at 144.7717 85.725 0)
+    (property "Value" "74HC132" (at 144.7717 85.725 0)
       (effects (font (size 1.27 1.27)))
     )
@@
       (effects (font (size 1.27 1.27)) (justify left))
     )
-    (property "Value" "74LS74" (at 110.5155 57.785 0)
+    (property "Value" "74HC74" (at 110.5155 57.785 0)
       (effects (font (size 1.27 1.27)) (justify left))
     )
@@
       (effects (font (size 1.27 1.27)) (justify left))
     )
-    (property "Value" "74LS74" (at 110.5155 97.79 0)
+    (property "Value" "74HC74" (at 110.5155 97.79 0)
       (effects (font (size 1.27 1.27)) (justify left))
     )
@@
       (effects (font (size 1.27 1.27)) (justify left))
     )
-    (property "Value" "74LS74" (at 110.5155 134.62 0)
+    (property "Value" "74HC74" (at 110.5155 134.62 0)
       (effects (font (size 1.27 1.27)) (justify left))
     )
@@
       (effects (font (size 1.27 1.27)) (justify left))
     )
-    (property "Value" "74LS74" (at 227.33 43.18 0)
+    (property "Value" "74HC74" (at 227.33 43.18 0)
       (effects (font (size 1.27 1.27)) (justify left))
     )
@@
       (effects (font (size 1.27 1.27)))
     )
-    (property "Value" "74LS132" (at 64.7617 46.99 0)
-      (effects (font (size 1.27 1.27)))
-    )
-    (property "Footprint" "" (at 64.77 52.705 0)
+    (property "Value" "74HC132" (at 64.7617 46.99 0)
+      (effects (font (size 1.27 1.27)))
+    )
+    (property "Footprint" "Package_DIP:DIP-14_W7.62mm_Socket" (at 64.77 52.705 0)
       (effects (font (size 1.27 1.27)) hide)
     )
@@
       (effects (font (size 1.27 1.27)))
     )
-    (property "Value" "74LS132" (at 86.3517 49.53 0)
-      (effects (font (size 1.27 1.27)))
-    )
-    (property "Footprint" "" (at 86.36 55.245 0)
+    (property "Value" "74HC132" (at 86.3517 49.53 0)
+      (effects (font (size 1.27 1.27)))
+    )
+    (property "Footprint" "Package_DIP:DIP-14_W7.62mm_Socket" (at 86.36 55.245 0)
       (effects (font (size 1.27 1.27)) hide)
     )
@@
       (effects (font (size 1.27 1.27)) (justify left))
     )
-    (property "Value" "74LS74" (at 110.5155 40.005 0)
-      (effects (font (size 1.27 1.27)) (justify left))
-    )
+    (property "Value" "74HC74" (at 110.5155 40.005 0)
+      (effects (font (size 1.27 1.27)) (justify left))
+    )
